File: EAGLE Files/Main/system_driver.brd (EAGLE design)
At the start: 53 x 66 mm, 27 parts

Commit message: Revised KIPR Board
Parts:
- added C1: (no value), rcl:C025-024X044
- PSOC: device ic-package:DIL28-4 -> ic-package:DIL28-3
- moved ICSP 2.84 mm to (34.3, 77.5)
- moved MISC 2.54 mm to (47.0, 72.4)
- moved J1 2.54 mm to (31.8, 30.5)
- moved J2 2.54 mm to (47.0, 30.5)
- moved PSOC 1.27 mm to (31.8, 21.6)
- moved REG5V 1.27 mm to (38.1, 59.7)
Connections:
- net GND: now also C1.2
- net VCC: now also C1.1
Routing:
- net MISC6: track 105.7 -> 63.2 mm, vias 0 -> 4
- net XRES: track 71.6 -> 112.7 mm, vias 0 -> 1
- net GND: track 69.9 -> 97.4 mm
- net MISC4: track 101.2 -> 74.9 mm, vias 0 -> 7
- net MISC3: track 86.2 -> 61.8 mm, vias 0 -> 3
- net VCC: track 123.5 -> 145.8 mm, vias 0 -> 6
- net RX: track 95.1 -> 117.1 mm, vias 1 -> 3
- net 3.3V: track 21.4 -> 0.00 mm
- net BO1: track 29.1 -> 48.4 mm
- net ENC2B: track 35.4 -> 53.1 mm, vias 1 -> 2
- net N$2: track 24.4 -> 38.9 mm, vias 0 -> 2
- net MISC1: track 96.9 -> 110.4 mm, vias 1 -> 0
- net MISC0: track 95.1 -> 107.6 mm
- net MISC2: track 82.7 -> 92.3 mm
- net AO2: track 35.8 -> 44.5 mm
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Other:
- board size 53 x 66 mm -> 53 x 67.3 mm
