File: EAGLE Files/Main/system_driver.sch (EAGLE design)
At the start: 27 parts

Commit message: Revised KIPR Board
Parts:
- added C1: (no value), rcl:C-US025-024X044
- PSOC: device ic-package:DIL28-4 -> ic-package:DIL28-3
Connections:
- net GND: now also C1.2
- net VCC: now also C1.1
Changed lines of the file:
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@@
 <?xml version="1.0" encoding="utf-8"?>
 <!DOCTYPE eagle SYSTEM "eagle.dtd">
-<eagle version="7.4.0">
+<eagle version="7.2.0">
 <drawing>
 <settings>
@@
 <part name="J1" library="SparkFun-Connectors" deviceset="M08" device="LONGPADS"/>
 <part name="J2" library="SparkFun-Connectors" deviceset="M08" device="LONGPADS"/>
-<part name="PSOC" library="ic-package" deviceset="DIL28" device="-4"/>
+<part name="PSOC" library="ic-package" deviceset="DIL28" device="-3"/>
 <part name="GND1" library="SparkFun-Aesthetics" deviceset="GND" device=""/>
 <part name="GND2" library="SparkFun-Aesthetics" deviceset="GND" device=""/>
@@
 <part name="GND19" library="SparkFun-Aesthetics" deviceset="GND" device=""/>
 <part name="VBAT4" library="supply2" deviceset="V+" device="" value="VBAT"/>
+<part name="C1" library="rcl" deviceset="C-US" device="025-024X044"/>
 </parts>
 <sheets>
@@
 <instance part="GND11" gate="1" x="-58.42" y="-27.94"/>
 <instance part="VBAT2" gate="1" x="-71.12" y="-15.24" rot="R90"/>
-<instance part="SUPPLY7" gate="G$1" x="-48.26" y="-15.24" rot="R270"/>
+<instance part="SUPPLY7" gate="G$1" x="-38.1" y="-15.24" rot="R270"/>
 <instance part="RX" gate="G$1" x="-109.22" y="12.7"/>
 <instance part="TX" gate="G$1" x="-119.38" y="12.7"/>
@@
 <instance part="GND19" gate="1" x="-111.76" y="-17.78"/>
 <instance part="VBAT4" gate="1" x="-111.76" y="-7.62"/>
+<instance part="C1" gate="G$1" x="-43.18" y="-20.32"/>
 </instances>
 <busses>
@@
 <pinref part="REG5V" gate="G$1" pin="OUT"/>
 <pinref part="SUPPLY7" gate="G$1" pin="VCC"/>
-<wire x1="-48.26" y1="-15.24" x2="-50.8" y2="-15.24" width="0.1524" layer="91"/>
+<wire x1="-38.1" y1="-15.24" x2="-43.18" y2="-15.24" width="0.1524" layer="91"/>
+<pinref part="C1" gate="G$1" pin="1"/>
+<wire x1="-43.18" y1="-15.24" x2="-50.8" y2="-15.24" width="0.1524" layer="91"/>
+<wire x1="-43.18" y1="-17.78" x2="-43.18" y2="-15.24" width="0.1524" layer="91"/>
+<junction x="-43.18" y="-15.24"/>
 </segment>
 <segment>
@@
 <pinref part="GND11" gate="1" pin="GND"/>
 <wire x1="-58.42" y1="-25.4" x2="-58.42" y2="-22.86" width="0.1524" layer="91"/>
-</segment>
-<segment>
+<pinref part="C1" gate="G$1" pin="2"/>
+<wire x1="-43.18" y1="-25.4" x2="-58.42" y2="-25.4" width="0.1524" layer="91"/>
+<junction x="-58.42" y="-25.4"/>
+</segment>
+<segment>
